Commit message: urdf 3 links

File: ROS2-urdf/install/servo6dof/share/servo6dof/urdf/servo6dof.urdf.xacro (robot description, xacro)
@@ -20,5 +20,5 @@
 	<link name="primeiro_elo">
 		<visual>
-			<origin rpy="0 0 0" xyz="0.25 0.55 0"/>
+			<origin rpy="0 0 0" xyz="0.25 0.57 0"/>
 			<geometry>
 				<mesh filename="package://servo6dof/meshes/manipulator_elo1.stl" scale="6 6 6"/>
@@ -30,5 +30,35 @@
 		<child link="primeiro_elo"/>
 		<axis xyz="0 0 1"/>
-		<origin rpy="0 0 -${PI/2}" xyz="0 -0.2 -0.01"/>
+		<origin rpy="0 0 -${PI/2}" xyz="0 -0.23 -0.01"/>
+		<limit lower="0" upper="${PI}" effort="${effort}" velocity="${velocity}"/>
+	</joint>
+	<link name="segundo_elo">
+		<visual>
+			<origin rpy="0 0 0" xyz="0.3 0.6 -0.55"/>
+			<geometry>
+				<mesh filename="package://servo6dof/meshes/manipulator_elo2.stl" scale="6 6 6"/>
+			</geometry>
+		</visual>
+	</link>
+	<joint name="joint_2" type="revolute">
+		<parent link="primeiro_elo"/>
+		<child link="segundo_elo"/>
+		<axis xyz="1 0 0"/>
+		<origin rpy="0 0 0" xyz="-0.05 -0.03 0.57"/>
+		<limit lower="-${PI/2}" upper="${PI/2}" effort="${effort}" velocity="${velocity}"/>
+	</joint>
+	<link name="terceiro_elo">
+		<visual>
+			<origin rpy="0 0 0" xyz="0.3 0.6 -0.55"/>
+			<geometry>
+				<mesh filename="package://servo6dof/meshes/manipulator_elo3.stl" scale="6 6 6"/>
+			</geometry>
+		</visual>
+	</link>
+	<joint name="joint_3" type="revolute">
+		<parent link="segundo_elo"/>
+		<child link="terceiro_elo"/>
+		<axis xyz="1 0 0"/>
+		<origin rpy="0 0 0" xyz="-0.05 -0.03 4"/>
 		<limit lower="-${PI/2}" upper="${PI/2}" effort="${effort}" velocity="${velocity}"/>
 	</joint>

File: ROS2-urdf/servo6dof/urdf/servo6dof.urdf.xacro (robot description, xacro)
@@ -20,5 +20,5 @@
 	<link name="primeiro_elo">
 		<visual>
-			<origin rpy="0 0 0" xyz="0.25 0.55 0"/>
+			<origin rpy="0 0 0" xyz="0.25 0.57 0"/>
 			<geometry>
 				<mesh filename="package://servo6dof/meshes/manipulator_elo1.stl" scale="6 6 6"/>
@@ -30,5 +30,35 @@
 		<child link="primeiro_elo"/>
 		<axis xyz="0 0 1"/>
-		<origin rpy="0 0 -${PI/2}" xyz="0 -0.2 -0.01"/>
+		<origin rpy="0 0 -${PI/2}" xyz="0 -0.23 -0.01"/>
+		<limit lower="0" upper="${PI}" effort="${effort}" velocity="${velocity}"/>
+	</joint>
+	<link name="segundo_elo">
+		<visual>
+			<origin rpy="0 0 0" xyz="0.3 0.6 -0.55"/>
+			<geometry>
+				<mesh filename="package://servo6dof/meshes/manipulator_elo2.stl" scale="6 6 6"/>
+			</geometry>
+		</visual>
+	</link>
+	<joint name="joint_2" type="revolute">
+		<parent link="primeiro_elo"/>
+		<child link="segundo_elo"/>
+		<axis xyz="1 0 0"/>
+		<origin rpy="0 0 0" xyz="-0.05 -0.03 0.57"/>
+		<limit lower="-${PI/2}" upper="${PI/2}" effort="${effort}" velocity="${velocity}"/>
+	</joint>
+	<link name="terceiro_elo">
+		<visual>
+			<origin rpy="0 0 0" xyz="0.25 0.6 -1.18"/>
+			<geometry>
+				<mesh filename="package://servo6dof/meshes/manipulator_elo3.stl" scale="6 6 6"/>
+			</geometry>
+		</visual>
+	</link>
+	<joint name="joint_3" type="revolute">
+		<parent link="segundo_elo"/>
+		<child link="terceiro_elo"/>
+		<axis xyz="1 0 0"/>
+		<origin rpy="0 0 0" xyz="0.06 0 0.63"/>
 		<limit lower="-${PI/2}" upper="${PI/2}" effort="${effort}" velocity="${velocity}"/>
 	</joint>

Commit message: garra_parcial

File: ROS2-urdf/install/servo6dof/share/servo6dof/urdf/servo6dof.urdf.xacro (robot description, xacro)
@@ -50,5 +50,5 @@
 	<link name="terceiro_elo">
 		<visual>
-			<origin rpy="0 0 0" xyz="0.3 0.6 -0.55"/>
+			<origin rpy="0 0 0" xyz="0.25 0.6 -1.18"/>
 			<geometry>
 				<mesh filename="package://servo6dof/meshes/manipulator_elo3.stl" scale="6 6 6"/>
@@ -60,5 +60,66 @@
 		<child link="terceiro_elo"/>
 		<axis xyz="1 0 0"/>
-		<origin rpy="0 0 0" xyz="-0.05 -0.03 4"/>
+		<origin rpy="0 0 0" xyz="0.06 0 0.63"/>
+		<limit lower="-${PI/2}" upper="${PI/2}" effort="${effort}" velocity="${velocity}"/>
+	</joint>
+	<link name="quarto_elo">
+		<visual>
+			<origin rpy="0 0 0" xyz="0.25 -0.187 -1.18"/>
+			<geometry>
+				<mesh filename="package://servo6dof/meshes/manipulator_elo4.stl" scale="6 6 6"/>
+			</geometry>
+		</visual>
+	</link>
+	<joint name="joint_4" type="revolute">
+		<parent link="terceiro_elo"/>
+		<child link="quarto_elo"/>
+		<axis xyz="1 0 0"/>
+		<origin rpy="0 0 0" xyz="0 0.78 0"/>
+		<limit lower="-${PI/2}" upper="${PI/2}" effort="${effort}" velocity="${velocity}"/>
+	</joint>
+	<link name="base_garra">
+		<visual>
+			<origin rpy="0 0 ${PI/2}" xyz="0 0 0"/>
+			<geometry>
+				<mesh filename="package://servo6dof/meshes/base_garra.stl" scale="6 6 6"/>
+			</geometry>
+		</visual>
+	</link>
+	<joint name="joint_5" type="revolute">
+		<parent link="quarto_elo"/>
+		<child link="base_garra"/>
+		<axis xyz="0 1 0"/>
+		<origin rpy="0 0 0" xyz="0.02 0.36 0"/>
+		<limit lower="-${PI/2}" upper="${PI/2}" effort="${effort}" velocity="${velocity}"/>
+	</joint>
+	<link name="garra_elo1">
+		<visual>
+			<origin rpy="0 ${PI} -${PI/2}" xyz="0.07 -0.15 0.05"/>
+			<geometry>
+				<mesh filename="package://servo6dof/meshes/garra_elo1.stl" scale="6 6 6"/>
+			</geometry>
+		</visual>
+	</link>
+	<joint name="joint_6" type="revolute">
+		<parent link="base_garra"/>
+		<child link="garra_elo1"/>
+		<axis xyz="0 0 1"/>
+		<origin rpy="0 0 0" xyz="-0.085 0.17 0.01"/>
+		<limit lower="-${PI/2}" upper="${PI/2}" effort="${effort}" velocity="${velocity}"/>
+	</joint>
+	<link name="garra_elo2a">
+		<visual>
+			<origin rpy="0 0 0" xyz="0 0 0"/>
+			<geometry>
+				<mesh filename="package://servo6dof/meshes/garra_elo2.stl" scale="6 6 6"/>
+			</geometry>
+		</visual>
+	</link>
+	<joint name="joint_garra_1" type="revolute">
+		<parent link="base_garra"/>
+		<child link="garra_elo2a"/>
+		<axis xyz="0 0 1"/>
+		<origin rpy="0 0 0" xyz="-0.085 0.4 0.01"/>
+		<mimic joint="joint_6" multiplier="1" offset="0" />
 		<limit lower="-${PI/2}" upper="${PI/2}" effort="${effort}" velocity="${velocity}"/>
 	</joint>

File: ROS2-urdf/servo6dof/urdf/servo6dof.urdf.xacro (robot description, xacro)
@@ -63,3 +63,64 @@
 		<limit lower="-${PI/2}" upper="${PI/2}" effort="${effort}" velocity="${velocity}"/>
 	</joint>
+	<link name="quarto_elo">
+		<visual>
+			<origin rpy="0 0 0" xyz="0.25 -0.187 -1.18"/>
+			<geometry>
+				<mesh filename="package://servo6dof/meshes/manipulator_elo4.stl" scale="6 6 6"/>
+			</geometry>
+		</visual>
+	</link>
+	<joint name="joint_4" type="revolute">
+		<parent link="terceiro_elo"/>
+		<child link="quarto_elo"/>
+		<axis xyz="1 0 0"/>
+		<origin rpy="0 0 0" xyz="0 0.78 0"/>
+		<limit lower="-${PI/2}" upper="${PI/2}" effort="${effort}" velocity="${velocity}"/>
+	</joint>
+	<link name="base_garra">
+		<visual>
+			<origin rpy="0 0 ${PI/2}" xyz="0 0 0"/>
+			<geometry>
+				<mesh filename="package://servo6dof/meshes/base_garra.stl" scale="6 6 6"/>
+			</geometry>
+		</visual>
+	</link>
+	<joint name="joint_5" type="revolute">
+		<parent link="quarto_elo"/>
+		<child link="base_garra"/>
+		<axis xyz="0 1 0"/>
+		<origin rpy="0 0 0" xyz="0.02 0.36 0"/>
+		<limit lower="-${PI/2}" upper="${PI/2}" effort="${effort}" velocity="${velocity}"/>
+	</joint>
+	<link name="garra_elo1">
+		<visual>
+			<origin rpy="0 ${PI} -${PI/2}" xyz="0.07 -0.15 0.05"/>
+			<geometry>
+				<mesh filename="package://servo6dof/meshes/garra_elo1.stl" scale="6 6 6"/>
+			</geometry>
+		</visual>
+	</link>
+	<joint name="joint_6" type="revolute">
+		<parent link="base_garra"/>
+		<child link="garra_elo1"/>
+		<axis xyz="0 0 1"/>
+		<origin rpy="0 0 0" xyz="-0.085 0.17 0.01"/>
+		<limit lower="-${PI/2}" upper="${PI/2}" effort="${effort}" velocity="${velocity}"/>
+	</joint>
+	<link name="garra_elo2a">
+		<visual>
+			<origin rpy="0 0 0" xyz="0 0 0"/>
+			<geometry>
+				<mesh filename="package://servo6dof/meshes/garra_elo2.stl" scale="6 6 6"/>
+			</geometry>
+		</visual>
+	</link>
+	<joint name="joint_garra_1" type="revolute">
+		<parent link="base_garra"/>
+		<child link="garra_elo2a"/>
+		<axis xyz="0 0 1"/>
+		<origin rpy="0 0 0" xyz="-0.085 0.4 0.01"/>
+		<mimic joint="joint_6" multiplier="1" offset="0" />
+		<limit lower="-${PI/2}" upper="${PI/2}" effort="${effort}" velocity="${velocity}"/>
+	</joint>
 </robot>

Commit message: finalizado (99%)

File: ROS2-urdf/install/servo6dof/share/servo6dof/urdf/servo6dof.urdf.xacro (robot description, xacro)
@@ -106,9 +106,9 @@
 		<axis xyz="0 0 1"/>
 		<origin rpy="0 0 0" xyz="-0.085 0.17 0.01"/>
-		<limit lower="-${PI/2}" upper="${PI/2}" effort="${effort}" velocity="${velocity}"/>
+		<limit lower="-${30*PI/180}" upper="${30*PI/180}" effort="${effort}" velocity="${velocity}"/>
 	</joint>
 	<link name="garra_elo2a">
 		<visual>
-			<origin rpy="0 0 0" xyz="0 0 0"/>
+			<origin rpy="0 0 0" xyz="-0.403 0.133 0"/>
 			<geometry>
 				<mesh filename="package://servo6dof/meshes/garra_elo2.stl" scale="6 6 6"/>
@@ -120,7 +120,23 @@
 		<child link="garra_elo2a"/>
 		<axis xyz="0 0 1"/>
-		<origin rpy="0 0 0" xyz="-0.085 0.4 0.01"/>
-		<mimic joint="joint_6" multiplier="1" offset="0" />
+		<origin rpy="0 0 0" xyz="-0.03 0.27 0.01"/>
+		<mimic joint="joint_6" multiplier="1" offset="-0.1" />
 		<limit lower="-${PI/2}" upper="${PI/2}" effort="${effort}" velocity="${velocity}"/>
 	</joint>
+	<link name="garra_elo3a">
+		<visual>
+			<origin rpy="0 ${PI} 0" xyz="0.28 0.205 0"/>
+			<geometry>
+				<mesh filename="package://servo6dof/meshes/garra_pinca.stl" scale="6 6 6"/>
+			</geometry>
+		</visual>
+	</link>
+	<joint name="joint_garra_2" type="revolute">
+		<parent link="garra_elo1"/>
+		<child link="garra_elo3a"/>
+		<axis xyz="0 0 1"/>
+		<origin rpy="0 0 -${PI/2}" xyz="-0.136 0.136 0"/>
+		<mimic joint="joint_6" multiplier="-0.1" offset="-0.3" />
+		<limit lower="0" upper="0.2" effort="${effort}" velocity="${velocity}"/>
+	</joint>
 </robot>

File: ROS2-urdf/servo6dof/urdf/servo6dof.urdf.xacro (robot description, xacro)
@@ -30,6 +30,6 @@
 		<child link="primeiro_elo"/>
 		<axis xyz="0 0 1"/>
-		<origin rpy="0 0 -${PI/2}" xyz="0 -0.23 -0.01"/>
-		<limit lower="0" upper="${PI}" effort="${effort}" velocity="${velocity}"/>
+		<origin rpy="0 0 0" xyz="0 -0.23 -0.01"/>
+		<limit lower="-${PI/2}" upper="${PI/2}" effort="${effort}" velocity="${velocity}"/>
 	</joint>
 	<link name="segundo_elo">
@@ -105,10 +105,10 @@
 		<child link="garra_elo1"/>
 		<axis xyz="0 0 1"/>
-		<origin rpy="0 0 0" xyz="-0.085 0.17 0.01"/>
-		<limit lower="-${PI/2}" upper="${PI/2}" effort="${effort}" velocity="${velocity}"/>
+		<origin rpy="0 0 0" xyz="-0.072 0.12 0.01"/>
+		<limit lower="-${40*PI/180}" upper="${30*PI/180}" effort="${effort}" velocity="${velocity}"/>
 	</joint>
 	<link name="garra_elo2a">
 		<visual>
-			<origin rpy="0 0 0" xyz="0 0 0"/>
+			<origin rpy="0 0 0" xyz="-0.403 0.133 0"/>
 			<geometry>
 				<mesh filename="package://servo6dof/meshes/garra_elo2.stl" scale="6 6 6"/>
@@ -120,7 +120,71 @@
 		<child link="garra_elo2a"/>
 		<axis xyz="0 0 1"/>
-		<origin rpy="0 0 0" xyz="-0.085 0.4 0.01"/>
-		<mimic joint="joint_6" multiplier="1" offset="0" />
+		<origin rpy="0 0 0" xyz="-0.05 0.27 0.01"/>
+		<mimic joint="joint_6" multiplier="1" offset="-0.2" />
 		<limit lower="-${PI/2}" upper="${PI/2}" effort="${effort}" velocity="${velocity}"/>
 	</joint>
+	<link name="garra_elo3a">
+		<visual>
+			<origin rpy="0 ${PI} 0" xyz="0.28 0.205 0"/>
+			<geometry>
+				<mesh filename="package://servo6dof/meshes/garra_pinca.stl" scale="6 6 6"/>
+			</geometry>
+		</visual>
+	</link>
+	<joint name="joint_pinca_a" type="revolute">
+		<parent link="garra_elo1"/>
+		<child link="garra_elo3a"/>
+		<axis xyz="0 0 1"/>
+		<origin rpy="0 0 -${PI/2}" xyz="-0.13 0.13 0"/>
+		<mimic joint="joint_6" multiplier="-1" offset="0.2" />
+		<limit effort="${effort}" velocity="${velocity}"/>
+	</joint>
+	<link name="garra_elo2">
+		<visual>
+			<origin rpy="0 0 ${PI/2}" xyz="-0.07 -0.15 -0.03"/>
+			<geometry>
+				<mesh filename="package://servo6dof/meshes/garra_elo1.stl" scale="6 6 6"/>
+			</geometry>
+		</visual>
+	</link>
+	<joint name="joint_7" type="revolute">
+		<parent link="base_garra"/>
+		<child link="garra_elo2"/>
+		<axis xyz="0 0 1"/>
+		<origin rpy="0 0 0" xyz="+0.072 0.12 0.01"/>
+		<mimic joint="joint_6" multiplier="-1" offset="0" />
+		<limit lower="-${30*PI/180}" upper="${30*PI/180}" effort="${effort}" velocity="${velocity}"/>
+	</joint>
+	<link name="garra_elo2b">
+		<visual>
+			<origin rpy="0 0 ${PI}" xyz="0.273 -0.036 0"/>
+			<geometry>
+				<mesh filename="package://servo6dof/meshes/garra_elo2.stl" scale="6 6 6"/>
+			</geometry>
+		</visual>
+	</link>
+	<joint name="joint_garra_3" type="revolute">
+		<parent link="base_garra"/>
+		<child link="garra_elo2b"/>
+		<axis xyz="0 0 1"/>
+		<origin rpy="0 0 0" xyz="+0.04 0.27 0.01"/>
+		<mimic joint="joint_6" multiplier="-1" offset="-1.6708" />
+		<limit lower="-${PI/2}" upper="${PI/2}" effort="${effort}" velocity="${velocity}"/>
+	</joint>
+	<link name="garra_elo3b">
+		<visual>
+			<origin rpy="0 0 0" xyz="-0.285 0.205 0"/>
+			<geometry>
+				<mesh filename="package://servo6dof/meshes/garra_pinca.stl" scale="6 6 6"/>
+			</geometry>
+		</visual>
+	</link>
+	<joint name="joint_pinca_b" type="revolute">
+		<parent link="garra_elo2"/>
+		<child link="garra_elo3b"/>
+		<axis xyz="0 0 1"/>
+		<origin rpy="0 0 ${PI/2}" xyz="0.13 0.13 0"/>
+		<mimic joint="joint_6" multiplier="1" offset="-0.2" />
+		<limit effort="${effort}" velocity="${velocity}"/>
+	</joint>
 </robot>
