Commit message: last update

File: servo6dof/install/servo6dof_description/share/servo6dof_description/urdf/servo6dof.urdf.xacro (robot description, xacro)
@@ -4,6 +4,24 @@
 	<xacro:property name="effort" value="30.0"/>
 	<xacro:property name="velocity" value="10.0"/>
+	<xacro:macro name="default_inertial" params="mass">
+		<inertial>
+			<mass value = "${mass}"/>
+			<inertia ixx="1.0" ixy="0.0" ixz="0.0"
+					 iyy="1.0" iyz="0.0"
+					 izz="1.0"/>
+		</inertial>
+	</xacro:macro>
+	<xacro:macro name="default_transmission" params="number">
+		<transmission name="transmission_${number}">
+			<plugin>transmission_interface/SimpleTransmission</plugin>
+			<actuator name="motor_${number}" role="acuator1"/>
+			<joint name="joint_${number}" role="joint1">
+				<mechanical_reduction>1.0</mechanical_reduction>
+			</joint>
+		</transmission>
+	</xacro:macro>
 	<link name="world"/>
 	<link name="base_link">
+		<xacro:default_inertial mass="1.0"/>
 		<visual>
 			<origin rpy="0 0 0" xyz="0.25 0.25 0"/>
@@ -12,4 +30,10 @@
 			</geometry>
 		</visual>
+		<collision>
+			<origin rpy="0 0 0" xyz="0.25 0.25 0"/>
+			<geometry>
+				<mesh filename="package://servo6dof_description/meshes/basement.stl" scale="6 6 6"/>
+			</geometry>
+		</collision>
 	</link>
 	<joint name="virtual_joint" type="fixed">
@@ -19,4 +43,5 @@
 	</joint>
 	<link name="primeiro_elo">
+		<xacro:default_inertial mass="0.1"/>
 		<visual>
 			<origin rpy="0 0 0" xyz="0.25 0.57 0"/>
@@ -25,4 +50,10 @@
 			</geometry>
 		</visual>
+		<collision>
+			<origin rpy="0 0 0" xyz="0.25 0.57 0"/>
+			<geometry>
+				<mesh filename="package://servo6dof_description/meshes/manipulator_elo1.stl" scale="6 6 6"/>
+			</geometry>
+		</collision>
 	</link>
 	<joint name="joint_1" type="revolute">
@@ -34,4 +65,5 @@
 	</joint>
 	<link name="segundo_elo">
+		<xacro:default_inertial mass="0.1"/>
 		<visual>
 			<origin rpy="0 0 0" xyz="0.3 0.6 -0.55"/>
@@ -40,4 +72,10 @@
 			</geometry>
 		</visual>
+		<collision>
+			<origin rpy="0 0 0" xyz="0.3 0.6 -0.55"/>
+			<geometry>
+				<mesh filename="package://servo6dof_description/meshes/manipulator_elo2.stl" scale="6 6 6"/>
+			</geometry>
+		</collision>
 	</link>
 	<joint name="joint_2" type="revolute">
@@ -49,4 +87,5 @@
 	</joint>
 	<link name="terceiro_elo">
+		<xacro:default_inertial mass="0.1"/>
 		<visual>
 			<origin rpy="0 0 0" xyz="0.25 0.6 -1.18"/>
@@ -55,4 +94,10 @@
 			</geometry>
 		</visual>
+		<collision>
+			<origin rpy="0 0 0" xyz="0.25 0.6 -1.18"/>
+			<geometry>
+				<mesh filename="package://servo6dof_description/meshes/manipulator_elo3.stl" scale="6 6 6"/>
+			</geometry>
+		</collision>
 	</link>
 	<joint name="joint_3" type="revolute">
@@ -64,4 +109,5 @@
 	</joint>
 	<link name="quarto_elo">
+		<xacro:default_inertial mass="0.1"/>
 		<visual>
 			<origin rpy="0 0 0" xyz="0.25 -0.187 -1.18"/>
@@ -70,4 +116,10 @@
 			</geometry>
 		</visual>
+		<collision>
+			<origin rpy="0 0 0" xyz="0.25 -0.187 -1.18"/>
+			<geometry>
+				<mesh filename="package://servo6dof_description/meshes/manipulator_elo4.stl" scale="6 6 6"/>
+			</geometry>
+		</collision>
 	</link>
 	<joint name="joint_4" type="revolute">
@@ -79,4 +131,5 @@
 	</joint>
 	<link name="base_garra">
+		<xacro:default_inertial mass="0.05"/>
 		<visual>
 			<origin rpy="0 0 ${PI/2}" xyz="0 0 0"/>
@@ -85,4 +138,10 @@
 			</geometry>
 		</visual>
+		<collision>
+			<origin rpy="0 0 ${PI/2}" xyz="0 0 0"/>
+			<geometry>
+				<mesh filename="package://servo6dof_description/meshes/base_garra.stl" scale="6 6 6"/>
+			</geometry>
+		</collision>
 	</link>
 	<joint name="joint_5" type="revolute">
@@ -94,4 +153,5 @@
 	</joint>
 	<link name="garra_elo1">
+		<xacro:default_inertial mass="0.01"/>
 		<visual>
 			<origin rpy="0 ${PI} -${PI/2}" xyz="0.07 -0.15 0.05"/>
@@ -100,4 +160,10 @@
 			</geometry>
 		</visual>
+		<collision>
+			<origin rpy="0 ${PI} -${PI/2}" xyz="0.07 -0.15 0.05"/>
+			<geometry>
+				<mesh filename="package://servo6dof_description/meshes/garra_elo1.stl" scale="6 6 6"/>
+			</geometry>
+		</collision>
 	</link>
 	<joint name="joint_6" type="revolute">
@@ -109,4 +175,5 @@
 	</joint>
 	<link name="garra_elo2a">
+		<xacro:default_inertial mass="0.01"/>
 		<visual>
 			<origin rpy="0 0 0" xyz="-0.403 0.133 0"/>
@@ -115,4 +182,10 @@
 			</geometry>
 		</visual>
+		<collision>
+			<origin rpy="0 0 0" xyz="-0.403 0.133 0"/>
+			<geometry>
+				<mesh filename="package://servo6dof_description/meshes/garra_elo2.stl" scale="6 6 6"/>
+			</geometry>
+		</collision>
 	</link>
 	<joint name="joint_garra_1" type="revolute">
@@ -125,4 +198,5 @@
 	</joint>
 	<link name="garra_elo3a">
+		<xacro:default_inertial mass="0.01"/>
 		<visual>
 			<origin rpy="0 ${PI} 0" xyz="0.28 0.205 0"/>
@@ -131,4 +205,10 @@
 			</geometry>
 		</visual>
+		<collision>
+			<origin rpy="0 ${PI} 0" xyz="0.28 0.205 0"/>
+			<geometry>
+				<mesh filename="package://servo6dof_description/meshes/garra_pinca.stl" scale="6 6 6"/>
+			</geometry>
+		</collision>
 	</link>
 	<joint name="joint_pinca_a" type="revolute">
@@ -141,4 +221,5 @@
 	</joint>
 	<link name="garra_elo2">
+		<xacro:default_inertial mass="0.01"/>
 		<visual>
 			<origin rpy="0 0 ${PI/2}" xyz="-0.07 -0.15 -0.03"/>
@@ -147,4 +228,10 @@
 			</geometry>
 		</visual>
+		<collision>
+			<origin rpy="0 0 ${PI/2}" xyz="-0.07 -0.15 -0.03"/>
+			<geometry>
+				<mesh filename="package://servo6dof_description/meshes/garra_elo1.stl" scale="6 6 6"/>
+			</geometry>
+		</collision>
 	</link>
 	<joint name="joint_7" type="revolute">
@@ -157,4 +244,5 @@
 	</joint>
 	<link name="garra_elo2b">
+		<xacro:default_inertial mass="0.01"/>
 		<visual>
 			<origin rpy="0 0 ${PI}" xyz="0.273 -0.036 0"/>
@@ -163,4 +251,10 @@
 			</geometry>
 		</visual>
+		<collision>
+			<origin rpy="0 0 ${PI}" xyz="0.273 -0.036 0"/>
+			<geometry>
+				<mesh filename="package://servo6dof_description/meshes/garra_elo2.stl" scale="6 6 6"/>
+			</geometry>
+		</collision>
 	</link>
 	<joint name="joint_garra_3" type="revolute">
@@ -173,4 +267,5 @@
 	</joint>
 	<link name="garra_elo3b">
+		<xacro:default_inertial mass="0.01"/>
 		<visual>
 			<origin rpy="0 0 0" xyz="-0.285 0.205 0"/>
@@ -179,4 +274,10 @@
 			</geometry>
 		</visual>
+		<collision>
+			<origin rpy="0 0 0" xyz="-0.285 0.205 0"/>
+			<geometry>
+				<mesh filename="package://servo6dof_description/meshes/garra_pinca.stl" scale="6 6 6"/>
+			</geometry>
+		</collision>
 	</link>
 	<joint name="joint_pinca_b" type="revolute">
@@ -188,3 +289,9 @@
 		<limit effort="${effort}" velocity="${velocity}"/>
 	</joint>
+	<xacro:default_transmission number="1"/>
+	<xacro:default_transmission number="2"/>
+	<xacro:default_transmission number="3"/>
+	<xacro:default_transmission number="4"/>
+	<xacro:default_transmission number="5"/>
+	<xacro:default_transmission number="6"/>
 </robot>

Commit message: ros2_control working

File: servo6dof/install/servo6dof_description/share/servo6dof_description/urdf/servo6dof.urdf.xacro (robot description, xacro)
@@ -1,4 +1,7 @@
 <?xml version="1.0"?>
 <robot xmlns:xacro="http://www.ros.org/wiki/xacro" name="servo6dof_description">
+	<xacro:arg name="is_ignition" default="true"/>
+	<xacro:include filename="$(find servo6dof_description)/urdf/servo6dof_gazebo.xacro"/>
+	<xacro:include filename="$(find servo6dof_description)/urdf/servo6dof_ros2_control.xacro"/>
 	<xacro:property name="PI" value="3.14159"/>
 	<xacro:property name="effort" value="30.0"/>
@@ -12,13 +15,4 @@
 		</inertial>
 	</xacro:macro>
-	<xacro:macro name="default_transmission" params="number">
-		<transmission name="transmission_${number}">
-			<plugin>transmission_interface/SimpleTransmission</plugin>
-			<actuator name="motor_${number}" role="acuator1"/>
-			<joint name="joint_${number}" role="joint1">
-				<mechanical_reduction>1.0</mechanical_reduction>
-			</joint>
-		</transmission>
-	</xacro:macro>
 	<link name="world"/>
 	<link name="base_link">
@@ -289,9 +283,3 @@
 		<limit effort="${effort}" velocity="${velocity}"/>
 	</joint>
-	<xacro:default_transmission number="1"/>
-	<xacro:default_transmission number="2"/>
-	<xacro:default_transmission number="3"/>
-	<xacro:default_transmission number="4"/>
-	<xacro:default_transmission number="5"/>
-	<xacro:default_transmission number="6"/>
 </robot>

File: servo6dof/install/servo6dof_description/share/servo6dof_description/urdf/servo6dof_gazebo.xacro (robot description, xacro)
@@ -1,10 +1,18 @@
 <?xml version="1.0"?>
 <robot xmlns:xacro="http://www.ros.org/wiki/xacro" name="servo6dof">
-	<gazebo>>
-		<plugin filename="libgazebo_ros2_control.so" name="gazebo_ros2_control">
-			<robot_param>robot_description</robot_param>
-			<robot_param_node>robot_state_publisher</robot_param_node>
-			<parameters></parameters>
-		</plugin>
-	</gazebo>
+  <!-- ROS 2 Control -->
+  <gazebo>
+    <!-- ROS 2 Humble -->
+    <xacro:if value="$(arg is_ignition)">
+      <plugin filename="ign_ros2_control-system" name="ign_ros2_control::IgnitionROS2ControlPlugin">
+        <parameters>$(find servo6dof_controller)/config/servo6dof_controllers.yaml</parameters>
+      </plugin>
+    </xacro:if>
+    <!-- ROS 2 Iron or above -->
+    <xacro:unless value="$(arg is_ignition)">
+      <plugin filename="gz_ros2_control-system" name="gz_ros2_control::GazeboSimROS2ControlPlugin">
+        <parameters>$(find servo6dof_controller)/config/servo6dof_controllers.yaml</parameters>
+      </plugin>
+    </xacro:unless>
+  </gazebo>
 </robot>

File: servo6dof/install/servo6dof_description/share/servo6dof_description/urdf/servo6dof_ros2_control.xacro (robot description, xacro)
@@ -3,14 +3,60 @@
         <xacro:property name="PI" value="3.14159"/>
 	<ros2_control name="RobotSystem" type="system">
-		<hardware>
-			<plugin>gazebo_ros2_control/GazeboSystem</plugin>
-		</hardware>
+		<xacro:if value="$(arg is_ignition)">
+			<hardware>
+				<plugin>ign_ros2_control/IgnitionSystem</plugin>
+			</hardware>
+		</xacro:if>
+		<xacro:unless value="$(arg is_ignition)">
+			<hardware>
+				<plugin>gz_ros2_control/GazeboSimSystem</plugin>
+			</hardware>
+		</xacro:unless>
 		<joint name="joint_1">
 			<command_interface name="position">
-				<param name="min"></param>
-				<param name="max"></param>
+				<param name="min">-${PI/2}</param>
+				<param name="max">${PI/2}</param>
 			</command_interface>
 			<state_interface name="position"/>
 		</joint>
+		<joint name="joint_2">
+			<command_interface name="position">
+				<param name="min">-${PI/2}</param>
+				<param name="max">${PI/2}</param>
+			</command_interface>
+			<state_interface name="position"/>
+		</joint>
+		<joint name="joint_3">
+			<command_interface name="position">
+				<param name="min">-${PI/2}</param>
+				<param name="max">${PI/2}</param>
+			</command_interface>
+			<state_interface name="position"/>
+		</joint>
+		<joint name="joint_4">
+			<command_interface name="position">
+				<param name="min">-${PI/2}</param>
+				<param name="max">${PI/2}</param>
+			</command_interface>
+			<state_interface name="position"/>
+		</joint>
+		<joint name="joint_5">
+			<command_interface name="position">
+				<param name="min">-${PI/2}</param>
+				<param name="max">${PI/2}</param>
+			</command_interface>
+			<state_interface name="position"/>
+		</joint>
+		<joint name="joint_6">
+			<command_interface name="position">
+				<param name="min">-${40*PI/180}</param>
+				<param name="max">${30*PI/180}</param>
+			</command_interface>
+			<state_interface name="position"/>
+		</joint>
+		<joint name="joint_7">
+			<param name="mimic">joint_6</param>
+			<param name="multiplier">-1</param>
+		</joint>
 	</ros2_control>
 </robot>
